File: 02_Electronics/MovuinoShieldPressure_ESP32/MovuinoShieldPressure.kicad_pcb (KiCad board)
At the start: 2 copper layers, 10.5 x 33 mm, 6 parts, among them J1 DF12-36NOLEGS-FEMALE, J2 Rext, J3 DF12-36NOLEGS-MALE

Commit message: Pressure Shield ESP32
Parts:
- added U$8: LOGO_MOVUINOBOTTOM_11MM, MovuinoESP8266:LOGO-NoName_MOVUINO_BMP_11MM-TOP, F.Cu at (104.8, 57.2)
- J1: footprint Connector_Hirose:Hirose_DF12_DF12C3.0-36DS-0.5V_2x18_P0.50mm_Vertical -> MovuinoESP8266:DF12-36-DP-NL-noPad
- moved J2 0.85 mm to (104.0, 36.6)
- renumbered R1 to Rref
Routing:
- net Net-(J1-Pad2): track 1.72 -> 0.00 mm
- net /ADC: track 23.6 -> 25.1 mm
- net VCC: track 19.3 -> 18.4 mm
Other:
- board text added: "Pressure Shield v1.1 by Adrien Husson"
- board text removed: "Movuino pressure shield v1.0"
- board text removed: "Rext"
- board text removed: "designed by Adrien Husson"
