File: 02_Electronics/MovuinoShieldCapacitiveTouch/MovuinoShieldCapacitiveTouch.kicad_pcb (KiCad board)
At the start: 2 copper layers, 10 parts, among them J1 DF12_3.0_-36DP_Female, J2 DF12_3.0_-36DP_Male, J3 FH12-10S-0.5SH(55), J4 Conn_01x06_Male, U1 FT5316DME

Commit message: shield_v2 done
Parts:
- added U$8: LOGO_MOVUINOBOTTOM_11MM, MovuinoESP8266:LOGO_MOVUINO_BMP_11MM-BOTTOM, F.Cu at (57.5, 67.6)
- added U$8: LOGO_MOVUINOBOTTOM_11MM, MovuinoESP8266:LOGO_MOVUINO_BMP_11MM-BOTTOM, B.Cu at (57.5, 67.6)
- J2: moved to B.Cu
- moved J4 105.4 mm to (80.4, 72.1), turned to 180 degrees
- moved J1 93.3 mm to (66.5, 79.5)
- moved J2 86.7 mm to (66.5, 79.5)
- moved C2 83.4 mm to (73.0, 72.1), turned to 90 degrees
- moved C1 80.5 mm to (75.3, 58.5), turned to 90 degrees
- moved C3 78.2 mm to (70.0, 72.1), turned to 90 degrees
- moved C4 72.2 mm to (67.1, 72.1), turned to 90 degrees
- moved U1 68.4 mm to (67.8, 65.5)
- moved J3 62.3 mm to (66.9, 53.4), turned to 180 degrees
- moved R1 61.8 mm to (75.3, 54.7), turned to 90 degrees
Connections:
- U1 pad 35: VDDA -> VCC
Routing:
- net GND: track 0.00 -> 69.4 mm, vias 0 -> 2
- net VCC: track 0.00 -> 52.9 mm, vias 0 -> 4
- net SCL: track 0.00 -> 49.6 mm, vias 0 -> 1
- net SDA: track 0.00 -> 44.7 mm, vias 0 -> 2
- net TX2: track 0.00 -> 14.5 mm, vias 0 -> 2
- net TX4: track 0.00 -> 13.7 mm
- net TX1: track 0.00 -> 13.4 mm, vias 0 -> 2
- net TX3: track 0.00 -> 13.3 mm
- net VDDA: track 0.00 -> 11.2 mm
- net RX6: track 0.00 -> 7.37 mm
- net RX5: track 0.00 -> 7.33 mm
- net RX4: track 0.00 -> 7.29 mm
- net RX3: track 0.00 -> 7.25 mm
- net RX2: track 0.00 -> 7.21 mm
- net RX1: track 0.00 -> 7.17 mm
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Other:
- board outline added: 33 x 33 mm
- net class Default: clearance 0.2 -> 0.1; trace_width 0.25 -> 0.2
- rule trace_clearance: 0.2 -> 0.1
- board text added: "3.3V"
- board text added: "GND"
- board text added: "SCL"
- board text added: "SDA"
